Commit message: Updated model definition

File: wasp_gazebo/urdf/drone.gazebo.xacro (robot description, xacro)
@@ -10,65 +10,50 @@
     <kp value="10000000.0"/>
     <kd value="1.0"/>
+<!--     <material>Gazebo/Black</material> -->
+  </gazebo>
+  <!--   Correct rotor colours that are not parsed properly -->
+  <xacro:macro name="rotor_material_loop" params="indices:=^">
+    <xacro:if value="${indices}">
+      <xacro:property name="index" value="${indices.pop(0)}"/>
+      <gazebo reference="rotor_${index}">
+        <material>
+          <xacro:if value="${index == 0 or index == 3 or index == 4}">Gazebo/Blue</xacro:if>
+          <xacro:if value="${index == 1 or index == 2 or index == 5}">Gazebo/Red</xacro:if></material>
+      </gazebo>
+      <xacro:rotor_material_loop/>
+    </xacro:if>
+  </xacro:macro>
+  <xacro:rotor_material_loop indices="${list(indices)}"/>
+  <gazebo reference="nozzle_link">
+      <visual name="extruder">
+        <pose frame=''>0 0 -0.05 0 0 0</pose>
+          <geometry>
+            <sphere>
+              <radius>0.01</radius>
+            </sphere>
+          </geometry>
+          <plugin name="foamer" filename="libwasp_gazebo.so">
+            <particleSize>0.02</particleSize>
+          </plugin>
+        </visual>
+    <material>Gazebo/White</material>
   </gazebo>
   <gazebo>
-    <link name="$(arg model)/ground_truth/odometry_sensorgt_link">
-      <pose>0 0 0 0 -0 0</pose>
+    <link name='$(arg model)/imu_link'>
+      <pose>0 0 0 0 0 0</pose>
       <inertial>
-        <pose>0 0 0 0 -0 0</pose>
-        <mass>0.15</mass>
+        <pose>0 0 0 0 0 0</pose>
+        <mass>0.015</mass>
         <inertia>
-          <ixx>0.0001</ixx>
+          <ixx>1e-05</ixx>
           <ixy>0</ixy>
           <ixz>0</ixz>
-          <iyy>0.0002</iyy>
+          <iyy>1e-05</iyy>
           <iyz>0</iyz>
-          <izz>0.0002</izz>
+          <izz>1e-05</izz>
         </inertia>
       </inertial>
-      <self_collide>0</self_collide>
     </link>
-    <joint name="$(arg model)/ground_truth/odometry_sensorgt_joint" type="revolute">
-      <child>$(arg model)/ground_truth/odometry_sensorgt_link</child>
-      <parent>base_link</parent>
-      <axis>
-        <xyz>0 0 1</xyz>
-        <limit>
-          <lower>0</lower>
-          <upper>0</upper>
-          <effort>0</effort>
-          <velocity>0</velocity>
-        </limit>
-        <dynamics>
-          <damping>1.0</damping>
-        </dynamics>
-        <use_parent_model_frame>1</use_parent_model_frame>
-      </axis>
-      <physics>
-        <ode>
-          <implicit_spring_damper>1</implicit_spring_damper>
-        </ode>
-      </physics>
-    </joint>
-    <link name="$(arg model)/imu_link">
-      <inertial>
-        <pose>0 0 0 0 0 0</pose>
-        <mass>0.15</mass>
-        <inertia>
-          <ixx>0.00001</ixx>
-          <ixy>0</ixy>
-          <ixz>0</ixz>
-          <iyy>0.00001</iyy>
-          <iyz>0</iyz>
-          <izz>0.00001</izz>
-        </inertia>
-      </inertial>
-      <sensor name="imu_sensor" type="imu">
-        <pose>0 0 0 3.141593 0 0</pose>
-        <always_on>1</always_on>
-        <update_rate>1000.0</update_rate>
-      </sensor>
-      <self_collide>0</self_collide>
-    </link>
-    <joint name="$(arg model)/imu_joint" type="revolute">
+    <joint name='$(arg model)/imu_joint' type='revolute'>
       <child>$(arg model)/imu_link</child>
       <parent>base_link</parent>
@@ -88,97 +73,137 @@
       </axis>
     </joint>
-  </gazebo>
-  <xacro:macro name="rotor" params="indices:=^">
-    <xacro:if value="${indices}">
-      <xacro:property name="idx" value="${indices.pop(0)}"/>
-      <gazebo reference="rotor_${idx}">
-        <xacro:if value="${idx % 2 == 0}">
-          <material>Gazebo/Red</material>
-        </xacro:if>
-        <xacro:unless value="${idx % 2 == 0}">
-          <material>Gazebo/Blue</material>
-        </xacro:unless>
-        <self_collide>0</self_collide>
-      </gazebo>
-      <gazebo>
-        <plugin name="rotor_${idx}_blade_1" filename="libLiftDragPlugin.so">
-          <a0>0.3</a0>
-          <alpha_stall>1.4</alpha_stall>
-          <cla>4.2500</cla>
-          <cda>0.10</cda>
-          <cma>0.00</cma>
-          <cla_stall>-0.025</cla_stall>
-          <cda_stall>0.0</cda_stall>
-          <cma_stall>0.0</cma_stall>
-          <area>0.002</area>
-          <air_density>1.2041</air_density>
-          <cp>0.084 0 0</cp>
-          <forward>0 ${1 - 2 * (idx % 2)} 0</forward>
-          <upward>0 0 1</upward>
-          <link_name>$(arg model)::rotor_${idx}</link_name>
+    <!-- Comment this section to disable GPS -->
+    <include>
+      <uri>model://gps</uri>
+      <pose>0 0 0 0 0 0</pose>
+      <name>gps</name>
+    </include>
+    <joint name='gps_joint' type='fixed'>
+      <child>gps::link</child>
+      <parent>base_link</parent>
+    </joint>
+    <plugin name='rosbag' filename='libgazebo_multirotor_base_plugin.so'>
+      <robotNamespace></robotNamespace>
+      <linkName>base_link</linkName>
+      <rotorVelocitySlowdownSim>10</rotorVelocitySlowdownSim>
+    </plugin>
+    <xacro:macro name="rotor_plugin_loop" params="indices:=^">
+      <xacro:if value="${indices}">
+        <xacro:property name="index" value="${indices.pop(0)}"/>
+        <plugin name='rotor_plugin_${index}' filename='libgazebo_motor_model.so'>
+          <robotNamespace></robotNamespace>
+          <jointName>rotor_${index}_joint</jointName>
+          <linkName>rotor_${index}</linkName>
+          <turningDirection>
+            <xacro:if value="${index == 1 or index == 2 or index == 5}">ccw</xacro:if>
+            <xacro:if value="${index == 0 or index == 3 or index == 4}">cw</xacro:if>
+          </turningDirection>
+          <timeConstantUp>0.0125</timeConstantUp>
+          <timeConstantDown>0.025</timeConstantDown>
+          <maxRotVelocity>1500</maxRotVelocity>
+          <motorConstant>8.54858e-06</motorConstant>
+          <momentConstant>0.06</momentConstant>
+          <commandSubTopic>/gazebo/command/motor_speed</commandSubTopic>
+          <motorNumber>${5 - index}</motorNumber>
+          <rotorDragCoefficient>0.000806428</rotorDragCoefficient>
+          <rollingMomentCoefficient>1e-06</rollingMomentCoefficient>
+          <motorSpeedPubTopic>/motor_speed/${5 - index}</motorSpeedPubTopic>
+          <rotorVelocitySlowdownSim>10</rotorVelocitySlowdownSim>
         </plugin>
-        <plugin name="rotor_${idx}_blade_2" filename="libLiftDragPlugin.so">
-          <a0>0.3</a0>
-          <alpha_stall>1.4</alpha_stall>
-          <cla>4.2500</cla>
-          <cda>0.10</cda>
-          <cma>0.00</cma>
-          <cla_stall>-0.025</cla_stall>
-          <cda_stall>0.0</cda_stall>
-          <cma_stall>0.0</cma_stall>
-          <area>0.002</area>
-          <air_density>1.2041</air_density>
-          <cp>-0.084 0 0</cp>
-          <forward>0 ${2 * (idx % 2) - 1} 0</forward>
-          <upward>0 0 1</upward>
-          <link_name>$(arg model)::rotor_${idx}</link_name>
-        </plugin>
-      </gazebo>
-      <xacro:rotor/>
-    </xacro:if>
-  </xacro:macro>
-  <xacro:rotor indices="${list(indices)}"/>
-  <gazebo>
-    <plugin name="arducopter_plugin" filename="libArduPilotPlugin.so">
-      <fdm_addr>127.0.0.1</fdm_addr>
-      <fdm_port_in>9002</fdm_port_in>
-      <fdm_port_out>9003</fdm_port_out>
-      <!--
-            Require by APM :
-            Only change model and gazebo from XYZ to XY-Z coordinates
-        -->
-      <modelXYZToAirplaneXForwardZDown>0 0 0 3.141593 0 0</modelXYZToAirplaneXForwardZDown>
-      <gazeboXYZToNED>0 0 0 3.141593 0 0</gazeboXYZToNED>
-      <imuName>$(arg model)::$(arg model)/imu_link::imu_sensor</imuName>
-      <connectionTimeoutMaxCount>5</connectionTimeoutMaxCount>
-      <!--
-            incoming control command [0, 1]
-            so offset it by 0 to get [0, 1]
-            and divide max target by 1.
-            offset = 0
-            multiplier = 838 max rpm / 1 = 838
-          -->
-      <xacro:macro name="channel" params="indices:=^">
-        <xacro:if value="${indices}">
-          <xacro:property name="idx" value="${indices.pop(0)}"/>
-          <control channel="${idx}">
-            <type>VELOCITY</type>
-            <offset>0</offset>
-            <p_gain>0.20</p_gain>
-            <i_gain>0</i_gain>
-            <d_gain>0</d_gain>
-            <i_max>0</i_max>
-            <i_min>0</i_min>
-            <cmd_max>2.5</cmd_max>
-            <cmd_min>-2.5</cmd_min>
-            <jointName>$(arg model)::rotor_${idx}_joint</jointName>
-            <multiplier>${(1 - 2 * (idx % 2)) * 920}</multiplier>
-            <controlVelocitySlowdownSim>1</controlVelocitySlowdownSim>
-          </control>
-          <xacro:channel/>
-        </xacro:if>
-      </xacro:macro>
-      <xacro:channel indices="${list(indices)}"/>
-    </plugin>
+        <xacro:rotor_plugin_loop/>
+      </xacro:if>
+    </xacro:macro>
+    <xacro:rotor_plugin_loop indices="${list(indices)}"/>
+    <plugin name='groundtruth_plugin' filename='libgazebo_groundtruth_plugin.so'>
+      <robotNamespace/>
+    </plugin>
+    <plugin name='magnetometer_plugin' filename='libgazebo_magnetometer_plugin.so'>
+      <robotNamespace/>
+      <pubRate>100</pubRate>
+      <noiseDensity>0.0004</noiseDensity>
+      <randomWalk>6.4e-06</randomWalk>
+      <biasCorrelationTime>600</biasCorrelationTime>
+      <magTopic>/mag</magTopic>
+    </plugin>
+    <plugin name='barometer_plugin' filename='libgazebo_barometer_plugin.so'>
+      <robotNamespace/>
+      <pubRate>50</pubRate>
+      <baroTopic>/baro</baroTopic>
+    </plugin>
+    <plugin name='mavlink_interface' filename='libgazebo_mavlink_interface.so'>
+      <robotNamespace></robotNamespace>
+      <imuSubTopic>/imu</imuSubTopic>
+      <magSubTopic>/mag</magSubTopic>
+      <baroSubTopic>/baro</baroSubTopic>
+      <mavlink_addr>INADDR_ANY</mavlink_addr>
+      <mavlink_tcp_port>4560</mavlink_tcp_port>
+      <mavlink_udp_port>14560</mavlink_udp_port>
+      <serialEnabled>0</serialEnabled>
+      <serialDevice>/dev/ttyACM0</serialDevice>
+      <baudRate>921600</baudRate>
+      <qgc_addr>INADDR_ANY</qgc_addr>
+      <qgc_udp_port>14550</qgc_udp_port>
+      <sdk_addr>INADDR_ANY</sdk_addr>
+      <sdk_udp_port>14540</sdk_udp_port>
+      <hil_mode>0</hil_mode>
+      <hil_state_level>false</hil_state_level>
+      <enable_lockstep>true</enable_lockstep>
+      <use_tcp>true</use_tcp>
+      <motorSpeedCommandPubTopic>/gazebo/command/motor_speed</motorSpeedCommandPubTopic>
+      <control_channels>
+        <xacro:macro name="rotor_channel_loop" params="indices:=^">
+          <xacro:if value="${indices}">
+            <xacro:property name="index" value="${indices.pop(0)}"/>
+            <channel name="rotor${index}">
+              <input_index>${index}</input_index>
+              <input_offset>0</input_offset>
+              <input_scaling>1500</input_scaling>
+              <zero_position_disarmed>0</zero_position_disarmed>
+              <zero_position_armed>100</zero_position_armed>
+              <joint_control_type>velocity</joint_control_type>
+            </channel>
+            <xacro:rotor_channel_loop/>
+          </xacro:if>
+        </xacro:macro>
+        <xacro:rotor_channel_loop indices="${list(indices)}"/>
+      </control_channels>
+    </plugin>
+    <plugin name='gazebo_imu_plugin' filename='libgazebo_imu_plugin.so'>
+      <robotNamespace></robotNamespace>
+      <linkName>$(arg model)/imu_link</linkName>
+      <imuTopic>/imu</imuTopic>
+      <gyroscopeNoiseDensity>0.0003394</gyroscopeNoiseDensity>
+      <gyroscopeRandomWalk>3.8785e-05</gyroscopeRandomWalk>
+      <gyroscopeBiasCorrelationTime>1000.0</gyroscopeBiasCorrelationTime>
+      <gyroscopeTurnOnBiasSigma>0.0087</gyroscopeTurnOnBiasSigma>
+      <accelerometerNoiseDensity>0.004</accelerometerNoiseDensity>
+      <accelerometerRandomWalk>0.006</accelerometerRandomWalk>
+      <accelerometerBiasCorrelationTime>300.0</accelerometerBiasCorrelationTime>
+      <accelerometerTurnOnBiasSigma>0.196</accelerometerTurnOnBiasSigma>
+    </plugin>
+    <!--    <plugin name='camera' filename='librealsense_gazebo_plugin.so'>
+      <prefix>camera</prefix>
+      <depthUpdateRate>30.0</depthUpdateRate>
+      <colorUpdateRate>30.0</colorUpdateRate>
+      <infraredUpdateRate>30.0</infraredUpdateRate>
+      <depthTopicName>depth/image_raw</depthTopicName>
+      <depthCameraInfoTopicName>depth/camera_info</depthCameraInfoTopicName>
+      <colorTopicName>color/image_raw</colorTopicName>
+      <colorCameraInfoTopicName>color/camera_info</colorCameraInfoTopicName>
+      <infrared1TopicName>infra1/image_raw</infrared1TopicName>
+      <infrared1CameraInfoTopicName>infra1/camera_info</infrared1CameraInfoTopicName>
+      <infrared2TopicName>infra2/image_raw</infrared2TopicName>
+      <infrared2CameraInfoTopicName>infra2/camera_info</infrared2CameraInfoTopicName>
+      <colorOpticalframeName>camera_color_optical_frame</colorOpticalframeName>
+      <depthOpticalframeName>camera_depth_optical_frame</depthOpticalframeName>
+      <infrared1OpticalframeName>camera_left_ir_optical_frame</infrared1OpticalframeName>
+      <infrared2OpticalframeName>camera_right_ir_optical_frame</infrared2OpticalframeName>
+      <rangeMinDepth>0.2</rangeMinDepth>
+      <rangeMaxDepth>10.0</rangeMaxDepth>
+      <pointCloud>1</pointCloud>
+      <pointCloudTopicName>depth/color/points</pointCloudTopicName>
+      <pointCloudCutoff>0.25</pointCloudCutoff>
+      <pointCloudCutoffMax>9.0</pointCloudCutoffMax>
+    </plugin>-->
   </gazebo>
 </robot>

File: wasp_gazebo/urdf/drone.urdf.xacro (robot description, xacro)
@@ -1,11 +1,11 @@
 <?xml version="1.0"?>
 <robot name="wasp" xmlns:xacro="http://www.ros.org/wiki/xacro">
-  <xacro:arg name="model" default="wasp" />
+ <xacro:arg name="model" default="wasp" />
   <xacro:include filename="$(find wasp_gazebo)/urdf/materials.xacro" />
   <xacro:include filename="$(find wasp_gazebo)/urdf/frame.xacro" />
-  <xacro:include filename="$(find wasp_gazebo)/urdf/drone.gazebo.xacro" />
-  <xacro:include filename="$(find realsense2_description)/urdf/_d435.urdf.xacro" />
-  <xacro:sensor_d435 name="camera" topics_ns="camera" parent="base_link" publish_pointcloud="true">
-    <origin xyz="0 -0.118 -0.074" rpy="0 ${pi/4} ${-pi/2}" />
-  </xacro:sensor_d435>
+  <xacro:include filename="$(find wasp_gazebo)/urdf/drone.gazebo.xacro"  />
+<!--  <xacro:include filename="$(find realsense2_description)/urdf/_d435.urdf.xacro" />
+  <xacro:sensor_d435 name="camera" topics_ns="camera" parent="base_link" publish_pointcloud="false">
+    <origin xyz="0 -0.070 -0.138" rpy="0 ${pi/2} ${-pi/2}" />
+  </xacro:sensor_d435>-->
 </robot>

File: wasp_gazebo/urdf/frame.xacro (robot description, xacro)
@@ -3,14 +3,14 @@
   <xacro:property name="mesh_path" value="package://wasp_gazebo/meshes/"/>
   <xacro:property name="r_a" value="0.075"/>
-  <xacro:property name="r_p" value="0.277"/>
-  <xacro:property name="r_l" value="0.092"/>
+  <xacro:property name="r_p" value="0.282"/>
+  <xacro:property name="r_l" value="0.074"/>
   <xacro:property name="del_p" value="${[0, pi, pi / 3, 4 * pi / 3, 2 * pi / 3, 5 * pi / 3]}"/>
-  <xacro:property name="del_l" value="${pi/6.2}"/>
-  <xacro:property name="idx" value="0"/>
+  <xacro:property name="del_l" value="${pi/5.9}"/>
+  <xacro:property name="index" value="0"/>
   <link name="base_link">
     <inertial>
-      <origin xyz="0 0 -0.05" rpy="0 0 0"/>
-      <mass value="1.6"/>
-      <inertia ixx="0.0177" ixy="0.0" ixz="0.0" iyy="0.016" iyz="0.0" izz="0.0025"/>
+      <origin xyz="0.00158 0.00084 -0.06501" rpy="0 0 0"/>
+      <mass value="3.67"/>
+      <inertia ixx="0.03" ixy="0.0" ixz="0.0" iyy="0.032" iyz="0.0" izz="0.0050"/>
     </inertial>
     <!--
@@ -29,5 +29,5 @@
     -->
     <collision name="lander">
-      <origin xyz="0 0 -0.08" rpy="0 0 0"/>
+      <origin xyz="0 0 -0.22" rpy="0 0 0"/>
       <geometry>
         <box size="0.3 0.2 0.16"/>
@@ -37,5 +37,23 @@
       <origin xyz="0 0 0" rpy="0 0 0"/>
       <geometry>
-        <mesh filename="${mesh_path}wasp_core.dae"/>
+        <mesh filename="${mesh_path}WASP_CORE.dae"/>
+      </geometry>
+    </visual>
+    <visual>
+      <origin xyz="0 0 0" rpy="0 0 0"/>
+      <geometry>
+        <mesh filename="${mesh_path}WASP_TOP.dae"/>
+      </geometry>
+    </visual>
+    <visual>
+      <origin xyz="0 0 -0.002" rpy="0 0 0"/>
+      <geometry>
+        <mesh filename="${mesh_path}WASP_CAGE.dae"/>
+      </geometry>
+    </visual>
+    <visual>
+      <origin xyz="0 0 -0.14" rpy="0 0 0"/>
+      <geometry>
+        <mesh filename="${mesh_path}WASP_EXTRUDER_MOUNT.dae"/>
       </geometry>
     </visual>
@@ -43,16 +61,16 @@
       <xacro:if value="${del_p}">
         <xacro:property name="theta" value="${del_p.pop(0)}"/>
-        <xacro:property name="idx" value="${6 - len(del_p)}"/>
-        <visual name="arm_${idx}">
-          <origin xyz="${r_a * cos(theta)} ${r_a * sin(theta)} 0.0125" rpy="0 0 ${theta + pi / 2}"/>
+        <xacro:property name="index" value="${6 - len(del_p)}"/>
+        <visual name="arm_${index}">
+          <origin xyz="${r_a * cos(theta)} ${r_a * sin(theta)} -0.0062" rpy="0 0 ${theta + pi / 2}"/>
           <geometry>
-            <mesh filename="${mesh_path}wasp_arm.dae"/>
+            <mesh filename="${mesh_path}WASP_ARM.dae"/>
           </geometry>
           <material name="black"/>
         </visual>
-        <visual name="motor_${idx}">
-          <origin xyz="${r_p * cos(theta)} ${r_p * sin(theta)} 0.0125" rpy="0 0 0"/>
+        <visual name="motor_${index}">
+          <origin xyz="${r_p * cos(theta)} ${r_p * sin(theta)} -0.0062" rpy="0 0 0"/>
           <geometry>
-            <mesh filename="${mesh_path}wasp_motor.dae"/>
+            <mesh filename="${mesh_path}WASP_MOTOR.dae"/>
           </geometry>
           <material name="black"/>
@@ -64,7 +82,7 @@
     <xacro:macro name="leg" params="prefix theta">
       <visual name="leg_${prefix}">
-        <origin xyz="${r_l * cos(theta)} ${r_l * sin(theta)} -0.063" rpy="0 0 ${theta + pi / 2}"/>
+        <origin xyz="${r_l * cos(theta)} ${r_l * sin(theta)} -0.206" rpy="0 0 ${theta + pi / 2}"/>
         <geometry>
-          <mesh filename="${mesh_path}wasp_leg.dae"/>
+          <mesh filename="${mesh_path}WASP_LEG.dae"/>
         </geometry>
         <material name="black"/>
@@ -76,15 +94,8 @@
     <xacro:leg prefix="3" theta="${pi - del_l}"/>
     <xacro:macro name="cargo" params="prefix reflect">
-      <visual name="rod_${prefix}">
-        <origin xyz="${0.037 * reflect} 0 -0.036" rpy="0 0 0"/>
+      <visual name="cannister_${prefix}">
+        <origin xyz="${0.08 * reflect} -0.076 -0.112" rpy="${-pi/2} 0 0"/>
         <geometry>
-          <mesh filename="${mesh_path}wasp_support_rod.dae"/>
-        </geometry>
-        <material name="black"/>
-      </visual>
-      <visual name="cannister_${prefix}">
-        <origin xyz="${0.063 * reflect} -0.076 -0.074" rpy="${-pi/2} 0 0"/>
-        <geometry>
-          <mesh filename="${mesh_path}wasp_cannister.dae"/>
+          <mesh filename="${mesh_path}WASP_CANNISTER.dae"/>
         </geometry>
         <material name="white"/>
@@ -94,16 +105,34 @@
     <xacro:cargo prefix="1" reflect="-1" />
   </link>
+  <link name="nozzle_link">
+    <inertial>
+      <origin xyz="0 0 0" rpy="0 0 0"/>
+      <mass value="0.01"/>
+      <inertia ixx="0.0001" ixy="0.0" ixz="0.0" iyy="0.0001" iyz="0.0" izz="0.0001"/>
+    </inertial>
+    <visual>
+      <origin xyz="0 0 0" rpy="0 0 ${pi/2}"/>
+      <geometry>
+        <mesh filename="${mesh_path}WASP_NOZZLE.dae"/>
+      </geometry>
+    </visual>
+  </link>
+  <joint name="nozzle_joint" type="fixed">
+    <parent link="base_link"/>
+    <child link="nozzle_link"/>
+    <origin xyz="-0.059 0.023 -0.286" rpy="0 0 0"/>
+  </joint>
   <xacro:macro name="rotor" params="del_p:=^">
     <xacro:if value="${del_p}">
       <xacro:property name="theta" value="${del_p.pop(0)}"/>
-      <xacro:property name="idx" value="${6 - len(del_p)}"/>
-      <joint name="rotor_${idx}_joint" type="continuous">
+      <xacro:property name="index" value="${6 - len(del_p)}"/>
+      <joint name="rotor_${index}_joint" type="continuous">
         <parent link="base_link"/>
-        <child link="rotor_${idx}"/>
-        <origin xyz="${r_p * cos(theta)} ${r_p * sin(theta)} 0.042" rpy="0 0 0"/>
+        <child link="rotor_${index}"/>
+        <origin xyz="${r_p * cos(theta)} ${r_p * sin(theta)} 0.029" rpy="0 0 0"/>
         <axis xyz="0 0 1"/>
         <dynamics damping="0.004"/>
       </joint>
-      <link name="rotor_${idx}">
+      <link name="rotor_${index}">
         <collision>
           <origin xyz="0 0 0" rpy="0 0 0"/>
@@ -119,16 +148,16 @@
         <visual>
           <origin xyz="0 0 0" rpy="0 0 0"/>
-          <xacro:if value="${idx % 2 == 0}">
+          <xacro:if value="${index == 0 or index == 3 or index == 4}">
             <geometry>
-              <mesh filename="${mesh_path}wasp_prop_cw.dae"/>
+              <mesh filename="${mesh_path}WASP_PROP_CW.dae"/>
+            </geometry>
+            <material name="blue"/>
+          </xacro:if>
+          <xacro:if value="${index == 1 or index == 2 or index == 5}">
+            <geometry>
+              <mesh filename="${mesh_path}WASP_PROP_CCW.dae"/>
             </geometry>
             <material name="red"/>
           </xacro:if>
-          <xacro:unless value="${idx % 2 == 0}">
-            <geometry>
-              <mesh filename="${mesh_path}wasp_prop_ccw.dae"/>
-            </geometry>
-            <material name="blue"/>
-          </xacro:unless>
         </visual>
       </link>

Commit message: Integration II

File: wasp_gazebo/urdf/drone.gazebo.xacro (robot description, xacro)
@@ -74,5 +74,5 @@
     </joint>
     <!-- Comment this section to disable GPS -->
-    <include>
+<!--    <include>
       <uri>model://gps</uri>
       <pose>0 0 0 0 0 0</pose>
@@ -82,5 +82,5 @@
       <child>gps::link</child>
       <parent>base_link</parent>
-    </joint>
+    </joint>-->
     <plugin name='rosbag' filename='libgazebo_multirotor_base_plugin.so'>
       <robotNamespace></robotNamespace>
