Commit message: VIO interface updates

File: wasp_gazebo/urdf/drone.gazebo.xacro (robot description, xacro)
@@ -74,5 +74,5 @@
     </joint>
     <!-- Comment this section to disable GPS -->
-<!--    <include>
+    <include>
       <uri>model://gps</uri>
       <pose>0 0 0 0 0 0</pose>
@@ -82,5 +82,5 @@
       <child>gps::link</child>
       <parent>base_link</parent>
-    </joint>-->
+    </joint>
     <plugin name='rosbag' filename='libgazebo_multirotor_base_plugin.so'>
       <robotNamespace></robotNamespace>

File: wasp_gazebo/urdf/drone.urdf (robot description, URDF)
Before this commit: robot wasp, 8 links, 7 joints
Links:
- link base_link: mass 3.67 -> 4.121

File: wasp_gazebo/urdf/frame.xacro (robot description, xacro)
@@ -11,5 +11,5 @@
     <inertial>
       <origin xyz="0.00158 0.00084 -0.06501" rpy="0 0 0"/>
-      <mass value="3.67"/>
+      <mass value="4.121"/>
       <inertia ixx="0.03" ixy="0.0" ixz="0.0" iyy="0.032" iyz="0.0" izz="0.0050"/>
     </inertial>

Commit message: Decoupled particle spawning from rendering loop

File: wasp_gazebo/urdf/drone.gazebo.xacro (robot description, xacro)
@@ -18,6 +18,6 @@
       <gazebo reference="rotor_${index}">
         <material>
-          <xacro:if value="${index == 0 or index == 3 or index == 4}">Gazebo/Blue</xacro:if>
-          <xacro:if value="${index == 1 or index == 2 or index == 5}">Gazebo/Red</xacro:if></material>
+          <xacro:if value="${index == 1 or index == 3 or index == 4}">Gazebo/Blue</xacro:if>
+          <xacro:if value="${index == 0 or index == 2 or index == 5}">Gazebo/Red</xacro:if></material>
       </gazebo>
       <xacro:rotor_material_loop/>
@@ -35,4 +35,5 @@
           <plugin name="foamer" filename="libwasp_gazebo.so">
             <particleSize>0.02</particleSize>
+            <divergence>7.18</divergence>
           </plugin>
         </visual>
@@ -96,6 +97,6 @@
           <linkName>rotor_${index}</linkName>
           <turningDirection>
-            <xacro:if value="${index == 1 or index == 2 or index == 5}">ccw</xacro:if>
-            <xacro:if value="${index == 0 or index == 3 or index == 4}">cw</xacro:if>
+            <xacro:if value="${index == 0 or index == 2 or index == 5}">ccw</xacro:if>
+            <xacro:if value="${index == 1 or index == 3 or index == 4}">cw</xacro:if>
           </turningDirection>
           <timeConstantUp>0.0125</timeConstantUp>
@@ -182,5 +183,5 @@
       <accelerometerTurnOnBiasSigma>0.196</accelerometerTurnOnBiasSigma>
     </plugin>
-    <!--    <plugin name='camera' filename='librealsense_gazebo_plugin.so'>
+<!--    <plugin name='camera' filename='librealsense_gazebo_plugin.so'>
       <prefix>camera</prefix>
       <depthUpdateRate>30.0</depthUpdateRate>

File: wasp_gazebo/urdf/drone.urdf (robot description, URDF)
Before this commit: robot wasp, 8 links, 7 joints
Links:
- link base_link: mass 4.121 -> 1.4121; geometry collision box size=0.3 0.2 0.16; collision cylinder length=0.09 radius=0.14
- link rotor_0: geometry collision cylinder length=0.01 radius=0.13; visual mesh filename=package://wasp_gazebo/meshes/WASP_PROP_CCW.dae
- link rotor_1: geometry collision cylinder length=0.01 radius=0.13; visual mesh filename=package://wasp_gazebo/meshes/WASP_PROP_CW.dae
Joints:
- joint rotor_0_joint: origin xyz=0.2794 0.0 0.029 rpy=0 0 0 -> xyz=-0.2794 3.42166315682e-17 0.029 rpy=0 0 0
- joint rotor_1_joint: origin xyz=-0.2794 3.42166315682e-17 0.029 rpy=0 0 0 -> xyz=0.2794 0.0 0.029 rpy=0 0 0
- joint rotor_2_joint: origin xyz=0.1397 0.241967497817 0.029 rpy=0 0 0 -> xyz=0.1397 -0.241967497817 0.029 rpy=0 0 0
- joint rotor_3_joint: origin xyz=-0.1397 -0.241967497817 0.029 rpy=0 0 0 -> xyz=-0.1397 0.241967497817 0.029 rpy=0 0 0
- joint rotor_4_joint: origin xyz=-0.1397 0.241967497817 0.029 rpy=0 0 0 -> xyz=-0.1397 -0.241967497817 0.029 rpy=0 0 0
- joint rotor_5_joint: origin xyz=0.1397 -0.241967497817 0.029 rpy=0 0 0 -> xyz=0.1397 0.241967497817 0.029 rpy=0 0 0

File: wasp_gazebo/urdf/frame.xacro (robot description, xacro)
@@ -5,11 +5,11 @@
   <xacro:property name="r_p" value="0.2794"/>
   <xacro:property name="r_l" value="0.074"/>
-  <xacro:property name="del_p" value="${[0, pi, pi / 3, 4 * pi / 3, 2 * pi / 3, 5 * pi / 3]}"/>
+  <xacro:property name="del_p" value="${[pi, 0, -pi / 3, 2 * pi / 3, 4 * pi / 3, pi / 3]}"/>
   <xacro:property name="del_l" value="${pi/5.9}"/>
   <xacro:property name="index" value="0"/>
-  <link name="base_link">
+  <link name="base_link" rpy="0 0 0">
     <inertial>
       <origin xyz="0.00158 0.00084 -0.06501" rpy="0 0 0"/>
-      <mass value="4.121"/>
+      <mass value="1.4121"/>
       <inertia ixx="0.03" ixy="0.0" ixz="0.0" iyy="0.032" iyz="0.0" izz="0.0050"/>
     </inertial>
@@ -21,11 +21,11 @@
       </geometry>
     </collision>
+    -->
     <collision name="rollcage">
-      <origin xyz="0 0 0.066" rpy="0 0 0"/>
+      <origin xyz="0 0 0.01" rpy="0 0 0"/>
       <geometry>
-        <cylinder length="0.06" radius="0.10"/>
+        <cylinder length="0.09" radius="0.14"/>
       </geometry>
     </collision>
-    -->
     <collision name="lander">
       <origin xyz="0 0 -0.22" rpy="0 0 0"/>
@@ -139,4 +139,5 @@
           <geometry>
             <cylinder length="0.01" radius="0.13"/>
+<!--             <box size="0.25 0.035 0.01"/> -->
           </geometry>
         </collision>
@@ -148,5 +149,5 @@
         <visual>
           <origin xyz="0 0 0" rpy="0 0 0"/>
-          <xacro:if value="${index == 0 or index == 3 or index == 4}">
+          <xacro:if value="${index == 1 or index == 3 or index == 4}">
             <geometry>
               <mesh filename="${mesh_path}WASP_PROP_CW.dae"/>
@@ -154,5 +155,5 @@
             <material name="blue"/>
           </xacro:if>
-          <xacro:if value="${index == 1 or index == 2 or index == 5}">
+          <xacro:if value="${index == 0 or index == 2 or index == 5}">
             <geometry>
               <mesh filename="${mesh_path}WASP_PROP_CCW.dae"/>
