Commit message: Update

File: wasp_gazebo/urdf/frame.xacro (robot description, xacro)
@@ -3,5 +3,5 @@
   <xacro:property name="mesh_path" value="package://wasp_gazebo/meshes/"/>
   <xacro:property name="r_a" value="0.075"/>
-  <xacro:property name="r_p" value="0.282"/>
+  <xacro:property name="r_p" value="0.2794"/>
   <xacro:property name="r_l" value="0.074"/>
   <xacro:property name="del_p" value="${[0, pi, pi / 3, 4 * pi / 3, 2 * pi / 3, 5 * pi / 3]}"/>

Commit message: Final update

File: wasp_gazebo/urdf/frame.xacro (robot description, xacro)
@@ -11,5 +11,5 @@
     <inertial>
       <origin xyz="0.00158 0.00084 -0.06501" rpy="0 0 0"/>
-      <mass value="1.4121"/>
+      <mass value="2.6121"/>
       <inertia ixx="0.03" ixy="0.0" ixz="0.0" iyy="0.032" iyz="0.0" izz="0.0050"/>
     </inertial>
